Commit message: slam_toolkit added

File: urdf/lidar.xacro (robot description, xacro)
@@ -2,5 +2,5 @@
 <robot xmlns:xacro="http://www.ros.org/wiki/xacro">
     <joint name="laser_joint" type="fixed">
-        <parent link="chassis" />
+        <parent link="base_link" />
         <child link="laser_frame" />
         <origin xyz="0.1 0 0.175" rpy="0 0 0" />
@@ -42,5 +42,5 @@
             </ray>
             <plugin name="gazebo_ros_laser" filename="libgazebo_ros_laser.so">
-                <topicName>/scan</topicName>
+                <topicName>scan</topicName>
                 <frameName>laser_frame</frameName>
             </plugin>

File: urdf/robot_core.xacro (robot description, xacro)
@@ -145,5 +145,5 @@
             <publishWheelTF>false</publishWheelTF>
             <publishOdomTF>true</publishOdomTF>
-            <publishWheelJointState>false</publishWheelJointState>
+            <publishWheelJointState>true</publishWheelJointState>
             <wheelAcceleration>0</wheelAcceleration>
             <wheelTorque>1</wheelTorque>
